File: Nova Mk I/Nova Mk I.kicad_sch (KiCad schematic)
At the start: 140 parts, among them J1 S2B-PH-K-SLFSN, J2 S2B-PH-K-SLFSN, J4 SJ-43516-SMT-TR, J5 SJ-43516-SMT-TR, J6 2171790001, SW1 SW_Push, SW10 SW_Push, SW11 SW_Push, SW12 SW_Push, SW13 SW_Push, SW14 SW_Push, SW15 SW_Push, SW16 SW_Push, SW17 SW_Push, SW18 SW_Push, SW19 SW_Push, SW2 SW_Push, SW20 SW_Push, SW21 SW_Push, SW3 SW_Push, SW4 SW_Push, SW5 SW_Push, SW6 SW_Push, SW7 SW_Push, SW8 SW_Push, SW9 SW_Push, U1 BQ24074RGTR, U3 USBLC6-2P6, U4 NRF52840-QIAA-R, X1 RT3215-32.768-12.5-TR, Y1 ECS-320-8-37B-CKY-TR

Commit message: Led changes
Parts:
- removed D22, D23, D24, D25, D26, D27, D28, D29, D30, D31, D32, D33, D34, D35, D36, D37, D38, D39, D40, D41, D42, D43, D44, D45, D46, D47, D48, D49, D50, D51, D52, D53, D54, D55, D56, D57, D58, D59, D60, D61, D62, D63: T36K3BGR-05D000121U1930, T36K3BGR-05D000121U1930:LED_T36K3BGR-05D000121U1930, symbol T36K3BGR-05D000121U1930:T36K3BGR-05D000121U1930
- removed Rgb_bl1, Rgb_gr1, Rgb_re1: R, symbol Device:R
- added Led1, Led10, Led11, Led12, Led13, Led14, Led15, Led16, Led17, Led18, Led19, Led2, Led20, Led21, Led3, Led4, Led5, Led6, Led7, Led8, Led9: ~, symbol LED_new:Led
- C12: value 1uF -> 100nF
- C14: value 100nF -> 1uF
- C16: value 1uF -> 47nF
- renumbered L5 to L1
Connections:
- new net: Led14. (VSS), Led15. (VSS), Led2. (VSS), Led3. (VSS), Led8. (VSS), Led9. (VSS)
- new net: Led1. (VSS), Led13. (VSS), Led14. (VSS), Led2. (VSS), Led7. (VSS), Led8. (VSS)
- new net: Led14. (VSS), Led8. (VSS)
- new net: Led2. (VSS), Led8. (VSS)
- new net: Led18. (VSS), Led21. (VSS)
- new net: Led11. (VSS), Led12. (VSS), Led17. (VSS), Led18. (VSS), Led20. (VSS), Led21. (VSS), Led5. (VSS), Led6. (VSS)
- new net: Led12. (VSS), Led18. (VSS), Led21. (VSS), Led6. (VSS)
- new net: Led20. (VSS), Led21. (VSS)
- new net: Led10. (VSS), Led15. (VSS), Led16. (VSS), Led19. (VSS), Led3. (VSS), Led4. (VSS), Led9. (VSS)
- new net: Led15. (VSS), Led9. (VSS)
- new net: Led3. (VSS), Led9. (VSS)
- new net: Led10. (VSS), Led4. (VSS)
- new net: Led10. (VSS), Led11. (VSS), Led16. (VSS), Led17. (VSS), Led19. (VSS), Led20. (VSS), Led4. (VSS), Led5. (VSS)
- new net: Led4. (VSS), Led5. (VSS)
- new net: Led13. (VSS), Led7. (VSS)
- new net: Led1. (VSS), Led13. (VSS), Led7. (VSS)
- new net: Led1. (VSS), Led7. (VSS)
- new net: Led13. (VSS), Led14. (VSS)
- new net: Led12. (VSS), Led18. (VSS)
- new net: Led12. (VSS), Led6. (VSS)
- new net: Led10. (VSS), Led16. (VSS)
- new net: Led17. (VSS), Led20. (VSS)
- new net: Led11. (VSS), Led5. (VSS)
- new net: Led11. (VSS), Led17. (VSS)
- new net: Led15. (VSS), Led19. (VSS)
- new net: Led16. (VSS), Led19. (VSS)
- new net: Led2. (VSS), Led3. (VSS)
- new net LED: Led1. (VSS)
Other:
- note removed: "LED's FIX RESISTOR"

Commit message: commit
Connections:
- net GND: now also Led1.3 (VSS), Led10.3 (VSS), Led11.3 (VSS), Led12.3 (VSS), Led13.3 (VSS), Led14.3 (VSS), Led15.3 (VSS), Led16.3 (VSS), Led17.3 (VSS), Led18.3 (VSS), Led19.3 (VSS), Led2.3 (VSS), Led20.3 (VSS), Led21.3 (VSS), Led3.3 (VSS), Led4.3 (VSS), Led5.3 (VSS), Led6.3 (VSS), Led7.3 (VSS), Led8.3 (VSS), Led9.3 (VSS), U1.5 (EN2); no longer J6.A1B12 (GND1), J6.B1A12 (GND2), U1.6 (EN1), U1.8 (VSS)
- net USB_D+: now also U4.B24 (XC1); no longer U4.AD6 (D+)
- net USB_D-: now also U4.A23 (XC2); no longer U4.AD4 (D-)
- net VBUS: now also U4.Y2 (VDDH); no longer J6.A4B9 (VBUS1), J6.B4A9 (VBUS2), U4.AD2 (VBUS)
- net VDD HV: now also U4.B3 (DCC); no longer U4.Y2 (VDDH)
- net at R15.2: now also J6.A6 (DP1); no longer J6.B5 (CC2)
- net at J6.B8 (SBU2): now also J6.B7 (DN2), R13.2
- net at L4.1: now also U4.AD2 (VBUS); no longer U4.AB2 (DCCH)
- net at C2.1, Y1.1 (IN/OUT): now also U4.H23 (ANT); no longer U4.A23 (XC2)
- net at C1.1, Y1.3 (OUT/IN): no longer U4.B24 (XC1)
- net at L2.2: now also U4.AB2 (DCCH); no longer U4.B3 (DCC)
- net at C3.1, L1.1: no longer U4.H23 (ANT)
- removed net LED: Led1. (VSS)
- new net: Led14.2 (DOUT), Led8.4 (DIN)
- new net: Led14.4 (DIN), Led15.2 (DOUT)
- new net: Led10.2 (DOUT), Led4.4 (DIN)
- new net: Led10.4 (DIN), Led16.2 (DOUT)
- new net: Led19.4 (DIN), Led20.2 (DOUT)
- new net: Led17.2 (DOUT), Led20.4 (DIN)
- new net: J6.B5 (CC2), J6.B6 (DP2), R1.2
- new net: Led13.4 (DIN), Led7.2 (DOUT)
- new net: Led1.2 (DOUT), Led7.4 (DIN)
- new net: Led12.4 (DIN), Led18.2 (DOUT)
- new net: Led18.4 (DIN), Led21.2 (DOUT)
- new net: Led16.4 (DIN), Led19.2 (DOUT)
- new net: Led3.2 (DOUT), Led9.4 (DIN)
- new net: Led3.4 (DIN), Led4.2 (DOUT)
- new net: Led11.2 (DOUT), Led17.4 (DIN)
- new net: Led11.4 (DIN), Led5.2 (DOUT)
- new net: Led5.4 (DIN), Led6.2 (DOUT)
- new net: Led15.4 (DIN), Led9.2 (DOUT)
- new net: Led12.2 (DOUT), Led6.4 (DIN)
- new net: Led2.4 (DIN), Led8.2 (DOUT)
- new net: Led1.4 (DIN), Led2.2 (DOUT)
- new net LED_in: Led21.4 (DIN)
- new net VDD: Led1.1 (VDD), Led10.1 (VDD), Led11.1 (VDD), Led12.1 (VDD), Led13.1 (VDD), Led14.1 (VDD), Led15.1 (VDD), Led16.1 (VDD), Led17.1 (VDD), Led18.1 (VDD), Led2.1 (VDD), Led20.1 (VDD), Led21.1 (VDD), Led3.1 (VDD), Led4.1 (VDD), Led5.1 (VDD), Led6.1 (VDD), Led7.1 (VDD), Led8.1 (VDD), Led9.1 (VDD)
- now unconnected: J6.A7 (DN1)
- no-connect marks 2 -> 3

Commit message: update
Parts:
- removed Led1, Led10, Led11, Led12, Led13, Led14, Led15, Led16, Led17, Led18, Led19, Led2, Led20, Led21, Led3, Led4, Led5, Led6, Led7, Led8, Led9: ~, symbol LED_new:Led
- added D22, D23, D24, D25, D26, D27, D28, D29, D30, D31, D32, D33, D34, D35, D36, D37, D38, D39, D40, D41, D42: SK6812-E, SK6812-E:LED_SK6812-E, symbol SK6812-E:SK6812-E
- added R7, R8: 4.7k, symbol Device:R
- added U2: ~, symbol yes:magnetic_connector
- renumbered L1 to L5
Connections:
- net GND: now also J6.A1B12 (GND1), J6.B1A12 (GND2), U1.6 (EN1), U1.8 (VSS), D22.3 (GND), D23.3 (GND), D24.3 (GND), D25.3 (GND), D26.3 (GND), D27.3 (GND), D28.3 (GND), D29.3 (GND), D30.3 (GND), D31.3 (GND), D32.3 (GND), D33.3 (GND), D34.3 (GND), D35.3 (GND), D36.3 (GND), D37.3 (GND), D38.3 (GND), D39.3 (GND), D40.3 (GND), D41.3 (GND), D42.3 (GND), U2. (Gnd); no longer U1.5 (EN2)
- net USB_D+: now also U4.AD6 (D+); no longer U4.B24 (XC1)
- net USB_D-: now also U4.AD4 (D-); no longer U4.A23 (XC2)
- net VBUS: now also J6.A4B9 (VBUS1), J6.B4A9 (VBUS2), U4.AD2 (VBUS), D22.1 (VDD), D23.1 (VDD), D24.1 (VDD), D25.1 (VDD), D26.1 (VDD), D27.1 (VDD), D28.1 (VDD), D29.1 (VDD), D30.1 (VDD), D31.1 (VDD), D32.1 (VDD), D33.1 (VDD), D34.1 (VDD), D35.1 (VDD), D36.1 (VDD), D37.1 (VDD), D38.1 (VDD), D39.1 (VDD), D40.1 (VDD), D41.1 (VDD), D42.1 (VDD); no longer U4.Y2 (VDDH)
- net VDD nRF: now also R7.2, R8.2, U2. (Gnd)
- net at J6.A6 (DP1): now also J6.B6 (DP2), R13.2; no longer R15.2
- net at J6.A7 (DN1): now also J6.B7 (DN2), R1.2
- net at L4.1: now also U4.AB2 (DCCH); no longer U4.AD2 (VBUS)
- net at C2.1, Y1.1 (IN/OUT): now also U4.A23 (XC2); no longer U4.H23 (ANT)
- net at L2.2: now also U4.B3 (DCC); no longer U4.AB2 (DCCH)
- net at C3.1, L5.1: now also U4.H23 (ANT)
- net at C1.1, Y1.3 (OUT/IN): now also U4.B24 (XC1)
- net RGB_BL: no longer names the net of U4.N1 (P0.08)
- net RGB_GR: no longer names the net of U4.M2 (P0.07/TRACECLK)
- net RGB_RE renamed LED
- net LED: now also D22.4 (DIN)
- net VDD HV renamed VLED
- net VLED: now also U4.Y2 (VDDH); no longer U4.B3 (DCC)
- new net: D31.2 (DOUT), D32.4 (DIN)
- new net: D30.2 (DOUT), D31.4 (DIN)
- new net: D36.2 (DOUT), D37.4 (DIN)
- new net: D35.2 (DOUT), D36.4 (DIN)
- new net: J6.B5 (CC2), R15.2
- new net: D37.2 (DOUT), D38.4 (DIN)
- new net: D40.2 (DOUT), D41.4 (DIN)
- new net: D39.2 (DOUT), D40.4 (DIN)
- new net: D23.2 (DOUT), D24.4 (DIN)
- new net: D22.2 (DOUT), D23.4 (DIN)
- new net: D29.2 (DOUT), D30.4 (DIN)
- new net: D27.2 (DOUT), D28.4 (DIN)
- new net: D26.2 (DOUT), D27.4 (DIN)
- new net: D33.2 (DOUT), D34.4 (DIN)
- new net: D32.2 (DOUT), D33.4 (DIN)
- new net: D25.2 (DOUT), D26.4 (DIN)
- new net: D24.2 (DOUT), D25.4 (DIN)
- new net: D28.2 (DOUT), D29.4 (DIN)
- new net: D38.2 (DOUT), D39.4 (DIN)
- new net: D41.2 (DOUT), D42.4 (DIN)
- new net: D34.2 (DOUT), D35.4 (DIN)
- new net Magnetic_data_1: R8.1, U2. (Gnd)
- new net Magnetic_data_2: R7.1, U2. (Gnd)
- now unconnected: J6.B8 (SBU2)
Other:
- note added: "LED's FIX RESISTOR"
- note added: "Magnetic"
- moved on the sheet: C17, C18, R3, X1

Commit message: footprints
Parts:
- removed J5: SJ-43516-SMT-TR, SJ-43516-SMT-TR:CUI_SJ-43516-SMT-TR, symbol SJ-43516-SMT-TR:SJ-43516-SMT-TR
- added R10, R16, R17, R9: 4.7k, Resistor_SMD:R_0402_1005Metric_Pad0.72x0.64mm_HandSolder, symbol Device:R
- C1, C10, C11, C12, C13, C14, C15, C16, C17, C18, C19, C2, C20, C21, C22, C23, C24, C26, C3, C4, C5, C6, C7, C8, C9: footprint (none) -> Capacitor_SMD:C_01005_0402Metric_Pad0.57x0.30mm_HandSolder
- CHG_LED1: footprint (none) -> LED_SMD:LED_0402_1005Metric_Pad0.77x0.64mm_HandSolder
- D22, D23, D24, D25, D26, D27, D28, D29, D30, D31, D32, D33, D34, D35, D36, D37, D38, D39, D40, D41, D42: footprint SK6812-E:LED_SK6812-E -> footprints:LED_SK6812-E
- J1, J2: footprint CONN_S2B-PH-K-S_JST -> footprints:CONN_S2B-PH-K-S_JST
- J4: footprint SJ-43516-SMT-TR:CUI_SJ-43516-SMT-TR -> footprints:trrs_new
- J6: footprint 2171790001:MOLEX_2171790001 -> footprints:USB
- L2, L4: footprint (none) -> Inductor_SMD:L_0603_1608Metric_Pad1.05x0.95mm_HandSolder
- L3, L5: footprint (none) -> Inductor_SMD:L_0402_1005Metric_Pad0.77x0.64mm_HandSolder
- PGOOD_LED1, R1, R11, R12, R13, R14, R15, R2, R3, R4, R5, R6, R7, R8: footprint (none) -> Resistor_SMD:R_0402_1005Metric_Pad0.72x0.64mm_HandSolder
- RESET_SW1: footprint (none) -> Button_Switch_SMD:SW_Push_1P1T_NO_E-Switch_TL3301NxxxxxG
- SW1, SW10, SW11, SW12, SW13, SW14, SW15, SW16, SW17, SW18, SW19, SW2, SW20, SW21, SW3, SW4, SW5, SW6, SW7, SW8, SW9: footprint (none) -> footprints:SW_PG1350_reversible
- U1: footprint BQ24074RGTR:QFN50P300X300X100-17N -> footprints:BATTERY_CHARGER
- U4: footprint NRF52840-QIAA-R:XCVR_NRF52840-QIAA-R -> footprints:MCU
- X1: footprint RT3215-32.768-12.5-TR:XTAL_RT3215-32.768-12.5-TR -> footprints:32kCrys
- Y1: footprint ECS-320-8-37B-CKY-TR:XTAL_ECS-160-9-37-CKM-TR -> footprints:32MHz_CRYSTAL
Connections:
- net DATA_CHAN_1: now also U4.W24 (P1.02), R10.2
- net DATA_CHAN_2: now also U4.V23 (P1.03), R9.2
- net Magnetic_data_1: now also U4.U24 (P1.04), R16.2
- net Magnetic_data_2: now also U4.T23 (P1.05), R17.2
- net VDD nRF: now also R10.1, R16.1, R17.1, R9.1
- net VLED renamed Vcc
